File: ring_light_controller.sch (KiCad schematic (older format))
At the start: 85 parts, among them J1 AudioJack2_Ground, J10 CHN_2_0, J11 CHN_2_1, J12 Color LED Port, J13 Conn_01x02, J2 CHAIN_IN, J3 CHAIN_OUT, J4 CHN_0_0, J5 CHN_0_1, J6 CHN_1_0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

Commit message: Updated footprints to work with JLCPCB assembly parts
Parts:
- L1: footprint Inductor_SMD:L_12x12mm_H6mm -> justb:L_SUNLORD_SWRB1205S_12.5x12.5mm_H6mm
- R17, R18, R23, R24, R30, R31: footprint Resistor_SMD:R_0603_1608Metric -> Resistor_SMD:R_1206_3216Metric
Changed lines of the file:
@@
 Sheet 1 1
 Title "Ring Light Controller v4"
-Date "2021-07-08"
-Rev "2"
+Date "2021-07-09"
+Rev "3"
 Comp "Brigham Young University HBLL"
 Comment1 ""
@@
 F 0 "R17" H 10518 6496 50  0000 L CNN
 F 1 "2.3" H 10518 6405 50  0000 L CNN
-F 2 "Resistor_SMD:R_0603_1608Metric" V 10490 6440 50  0001 C CNN
+F 2 "Resistor_SMD:R_1206_3216Metric" V 10490 6440 50  0001 C CNN
 F 3 "~" H 10450 6450 50  0001 C CNN
 F 4 "C247504" H 10450 6450 50  0001 C CNN "LCSC Part #"
@@
 F 0 "R23" H 12868 6496 50  0000 L CNN
 F 1 "2.3" H 12868 6405 50  0000 L CNN
-F 2 "Resistor_SMD:R_0603_1608Metric" V 12840 6440 50  0001 C CNN
+F 2 "Resistor_SMD:R_1206_3216Metric" V 12840 6440 50  0001 C CNN
 F 3 "~" H 12800 6450 50  0001 C CNN
 F 4 "C247504" H 12800 6450 50  0001 C CNN "LCSC Part #"
@@
 F 0 "R30" H 15168 6496 50  0000 L CNN
 F 1 "2.3" H 15168 6405 50  0000 L CNN
-F 2 "Resistor_SMD:R_0603_1608Metric" V 15140 6440 50  0001 C CNN
+F 2 "Resistor_SMD:R_1206_3216Metric" V 15140 6440 50  0001 C CNN
 F 3 "~" H 15100 6450 50  0001 C CNN
 F 4 "C247504" H 15100 6450 50  0001 C CNN "LCSC Part #"
@@
 F 0 "R18" H 10518 8546 50  0000 L CNN
 F 1 "2.3" H 10518 8455 50  0000 L CNN
-F 2 "Resistor_SMD:R_0603_1608Metric" V 10490 8490 50  0001 C CNN
+F 2 "Resistor_SMD:R_1206_3216Metric" V 10490 8490 50  0001 C CNN
 F 3 "~" H 10450 8500 50  0001 C CNN
 F 4 "C247504" H 10450 8500 50  0001 C CNN "LCSC Part #"
@@
 F 0 "R24" H 12868 8546 50  0000 L CNN
 F 1 "2.3" H 12868 8455 50  0000 L CNN
-F 2 "Resistor_SMD:R_0603_1608Metric" V 12840 8490 50  0001 C CNN
+F 2 "Resistor_SMD:R_1206_3216Metric" V 12840 8490 50  0001 C CNN
 F 3 "~" H 12800 8500 50  0001 C CNN
 F 4 "C247504" H 12800 8500 50  0001 C CNN "LCSC Part #"
@@
 F 0 "R31" H 15168 8546 50  0000 L CNN
 F 1 "2.3" H 15168 8455 50  0000 L CNN
-F 2 "Resistor_SMD:R_0603_1608Metric" V 15140 8490 50  0001 C CNN
+F 2 "Resistor_SMD:R_1206_3216Metric" V 15140 8490 50  0001 C CNN
 F 3 "~" H 15100 8500 50  0001 C CNN
 F 4 "C247504" H 15100 8500 50  0001 C CNN "LCSC Part #"
@@
 F 0 "L1" H 13600 3515 50  0000 C CNN
 F 1 "68uH" H 13600 3424 50  0000 C CNN
-F 2 "Inductor_SMD:L_12x12mm_H6mm" H 13600 3300 50  0001 C CNN
+F 2 "justb:L_SUNLORD_SWRB1205S_12.5x12.5mm_H6mm" H 13600 3300 50  0001 C CNN
 F 3 "~" H 13600 3300 50  0001 C CNN
 F 4 "C169388" H 13600 3300 50  0001 C CNN "LCSC Part #"
