File: ring_light_controller.kicad_pcb (KiCad board)
At the start: 2 copper layers, 81.9 x 82.6 mm, 85 parts, among them J1 AudioJack2_Ground, J10 CHN_2_0, J11 CHN_2_1, J12 Color LED Port, J13 Conn_01x02, J2 CHAIN_IN, J3 CHAIN_OUT, J4 CHN_0_0, J5 CHN_0_1, J6 CHN_1_0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

Commit message: updated connecters to 3.5mm, and made opto resistors smaller in value
Parts:
- J2: value CHAIN_IN -> AudioJack3; footprint Connector_JST:JST_XH_B3B-XH-AM_1x03_P2.50mm_Vertical -> justb:Jack_3.5mm_BOOMELE_C18594-SMT_Horizontal
- J3: value CHAIN_OUT -> AudioJack3; footprint Connector_JST:JST_XH_B3B-XH-AM_1x03_P2.50mm_Vertical -> justb:Jack_3.5mm_BOOMELE_C18594-SMT_Horizontal
- J9: footprint Connector_PinHeader_1.27mm:PinHeader_1x03_P1.27mm_Vertical -> Connector_PinHeader_2.54mm:PinHeader_1x03_P2.54mm_Vertical
- R10, R9: value 1k -> 200
- moved Q1 9.64 mm to (122.2, 114.8)
- moved R7 9.64 mm to (120.3, 111.6)
- moved R11 9.64 mm to (119.0, 114.2)
- moved J12 5.10 mm to (124.4, 138.2), turned to 180 degrees
- moved J3 4.93 mm to (103.1, 119.9), turned to 90 degrees
- moved J2 3.20 mm to (103.1, 106.7), turned to 90 degrees
- moved J10 2.73 mm to (177.8, 85.9), turned to 270 degrees
- moved J4 2.73 mm to (177.8, 121.4), turned to 270 degrees
- moved J6 2.73 mm to (177.8, 103.6), turned to 270 degrees
- moved J11 2.50 mm to (177.8, 77.2), turned to 270 degrees
- moved J5 2.50 mm to (177.8, 112.8), turned to 270 degrees
- moved J7 2.50 mm to (177.8, 95.0), turned to 270 degrees
- moved R27 2.50 mm to (143.8, 100.6)
- moved D1 1.14 mm to (145.5, 96.8)
- moved R1 1.14 mm to (143.6, 96.8)
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Connections:
- J10 pad 1: +24V -> Net-(J10-Pad1)
- J10 pad 2: Net-(J10-Pad2) -> +24V
- J11 pad 1: +24V -> Net-(J11-Pad1)
- J11 pad 2: Net-(J11-Pad2) -> +24V
- J12 pad 1: +5V -> C_LED_CTRL
- J12 pad 3: C_LED_CTRL -> +5V
- J4 pad 1: +24V -> Net-(J4-Pad1)
- J4 pad 2: Net-(J4-Pad2) -> +24V
- J5 pad 1: +24V -> Net-(J5-Pad1)
- J5 pad 2: Net-(J5-Pad2) -> +24V
- J6 pad 1: +24V -> Net-(J6-Pad1)
- J6 pad 2: Net-(J6-Pad2) -> +24V
- J7 pad 1: +24V -> Net-(J7-Pad1)
- J7 pad 2: Net-(J7-Pad2) -> +24V
- Q12 pad 3: Net-(J10-Pad2) -> Net-(J10-Pad1)
- Q13 pad 3: Net-(J11-Pad2) -> Net-(J11-Pad1)
- Q4 pad 3: Net-(J4-Pad2) -> Net-(J4-Pad1)
- Q5 pad 3: Net-(J5-Pad2) -> Net-(J5-Pad1)
- Q8 pad 3: Net-(J6-Pad2) -> Net-(J6-Pad1)
- Q9 pad 3: Net-(J7-Pad2) -> Net-(J7-Pad1)
Routing:
- net GND: track 131.8 -> 169.2 mm, vias 21 -> 20
- net LOAD_IN: track 38.7 -> 63.1 mm
- net TX: track 49.6 -> 38.2 mm
- net Net-(J7-Pad1): track 0.00 -> 7.51 mm
- net Net-(J5-Pad1): track 0.00 -> 7.51 mm
- net Net-(J11-Pad1): track 0.00 -> 7.51 mm
- net Net-(J1-PadT): track 16.7 -> 9.50 mm
- net +5V: track 210.0 -> 216.9 mm, vias 3 -> 4
- net Net-(J6-Pad1): track 0.00 -> 6.67 mm
- net Net-(J4-Pad1): track 0.00 -> 6.67 mm
- net Net-(J10-Pad1): track 0.00 -> 6.67 mm
- net Net-(J7-Pad2): track 6.39 -> 0.00 mm
- net Net-(J5-Pad2): track 6.39 -> 0.00 mm
- net Net-(J11-Pad2): track 6.39 -> 0.00 mm
- net Net-(J6-Pad2): track 5.37 -> 0.00 mm
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
Commit message: slight changes
Parts:
- added D10: Green, LED_SMD:LED_0603_1608Metric, F.Cu at (114.8, 110.2)
- added D11: Green, LED_SMD:LED_0603_1608Metric, F.Cu at (114.8, 123.4)
- added D9: Green, LED_SMD:LED_0603_1608Metric, F.Cu at (104.4, 96.0)
- added R34: 1k, Resistor_SMD:R_0402_1005Metric, F.Cu at (116.8, 123.4)
- added R6: 1k, Resistor_SMD:R_0603_1608Metric, F.Cu at (106.2, 96.0)
- added R8: 1k, Resistor_SMD:R_0402_1005Metric, F.Cu at (116.8, 110.2)
- added REF**: OSHW-Logo_5.7x6mm_SilkScreen, Symbol:OSHW-Logo_5.7x6mm_SilkScreen, F.Cu at (154.9, 135.6)
- added REF**: ESD-Logo_6.6x6mm_SilkScreen, Symbol:ESD-Logo_6.6x6mm_SilkScreen, F.Cu at (163.6, 135.6)
- added TP2: TestPoint, TestPoint:TestPoint_Pad_D1.0mm, F.Cu at (117.4, 107.7)
- added TP3: TestPoint, TestPoint:TestPoint_Pad_D1.0mm, F.Cu at (122.4, 124.0)
- added TP6: TestPoint, TestPoint:TestPoint_Pad_D1.0mm, F.Cu at (116.8, 88.9)
Routing:
- net +5V: track 216.9 -> 229.6 mm
- net RX: track 31.9 -> 42.3 mm
- net LOAD_IN: track 63.1 -> 71.0 mm
- net TX: track 38.2 -> 44.5 mm
- net +24V: track 151.4 -> 156.9 mm
- net GND: track 169.2 -> 172.1 mm, vias 20 -> 21
- net Net-(D9-Pad2): track 0.00 -> 2.49 mm
- net Net-(D11-Pad2): track 0.00 -> 2.15 mm
- net Net-(D10-Pad2): track 0.00 -> 2.15 mm
Other:
- board text added: "LOAD"
- board text added: "Ring Light Controller v1"
- board text removed: "Ring Light Controller v4"

Commit message: fixed opto pin outputs
Parts:
- removed REF**: OSHW-Logo_5.7x6mm_SilkScreen, Symbol:OSHW-Logo_5.7x6mm_SilkScreen
- removed REF**: ESD-Logo_6.6x6mm_SilkScreen, Symbol:ESD-Logo_6.6x6mm_SilkScreen
Connections:
- U2 pad 3: Net-(J1-PadG) -> Net-(J1-PadT)
- U2 pad 4: Net-(J1-PadT) -> Net-(J1-PadG)
- U3 pad 3: Net-(J1-PadG) -> Net-(J1-PadS)
- U3 pad 4: Net-(J1-PadS) -> Net-(J1-PadG)
Routing:
- net Net-(J1-PadT): track 9.50 -> 14.9 mm
- net Net-(J1-PadG): track 15.4 -> 17.5 mm, vias 2 -> 0
- net Net-(J1-PadS): track 22.4 -> 20.4 mm

Commit message: updated to latest
Parts:
- added R35: 1k, Resistor_SMD:R_0402_1005Metric, F.Cu at (156.0, 121.9)
- added R36: 1k, Resistor_SMD:R_0402_1005Metric, F.Cu at (156.0, 110.7)
- added R37: 1k, Resistor_SMD:R_0402_1005Metric, F.Cu at (156.0, 103.6)
- added R38: 1k, Resistor_SMD:R_0402_1005Metric, F.Cu at (156.5, 93.0)
- added R39: 1k, Resistor_SMD:R_0402_1005Metric, F.Cu at (156.0, 85.9)
- added R40: 1k, Resistor_SMD:R_0402_1005Metric, F.Cu at (155.4, 75.2)
- added REF**: ESD-Logo_6.6x6mm_SilkScreen, Symbol:ESD-Logo_6.6x6mm_SilkScreen, F.Cu at (163.1, 134.6)
- added REF**: OSHW-Logo_5.7x6mm_SilkScreen, Symbol:OSHW-Logo_5.7x6mm_SilkScreen, F.Cu at (154.9, 134.6)
Routing:
- net GND: track 172.1 -> 194.0 mm
- net CHN_0_CTRL: track 43.0 -> 51.8 mm
- net CHN_2_CTRL: track 79.4 -> 84.4 mm
- net CHN_1_CTRL: track 47.2 -> 51.8 mm
